Commit message: no default use mock, fix name with space

File: touch_description/ros2_control/touch.ros2_control.xacro (robot description, xacro)
@@ -1,5 +1,5 @@
 <?xml version="1.0"?>
 <robot xmlns:xacro="http://www.ros.org/wiki/xacro">
-  <xacro:macro name="touch_ros2_control" params="name use_mock_hardware:=^|true device_name:=^|left">
+  <xacro:macro name="touch_ros2_control" params="name use_mock_hardware device_name">
     <ros2_control name="${name}" type="system">
       <hardware>

File: touch_description/urdf/touch.urdf.xacro (robot description, xacro)
@@ -1,6 +1,6 @@
 <?xml version="1.0"?>
 <robot xmlns:xacro="http://www.ros.org/wiki/xacro" name="touch">
-  <xacro:arg name="use_mock_hardware" default="true"/>
-  <xacro:arg name="device_name" default="left"/>
+  <xacro:arg name="use_mock_hardware" default="false"/>
+  <xacro:arg name="device_name" default="Default Device"/>
   <xacro:include filename="$(find touch_description)/ros2_control/touch.ros2_control.xacro"/>
   <link name="touch_base"/>

Commit message: refactor description to real joints

File: touch_description/ros2_control/touch.ros2_control.xacro (robot description, xacro)
@@ -13,19 +13,90 @@
         </xacro:unless>
       </hardware>
-      <joint name="touch_x">
-        <command_interface name="effort"/>
-        <state_interface name="position"/>
-        <state_interface name="velocity"/>
+      <joint name="waist">
+        <state_interface name="position">
+          <param name="initial_value">0.0</param>
+        </state_interface>
+        <state_interface name="velocity">
+          <param name="initial_value">0.0</param>
+        </state_interface>
       </joint>
-      <joint name="touch_y">
-        <command_interface name="effort"/>
-        <state_interface name="position"/>
-        <state_interface name="velocity"/>
+      <joint name="shoulder">
+        <state_interface name="position">
+          <param name="initial_value">0.0</param>
+        </state_interface>
+        <state_interface name="velocity">
+          <param name="initial_value">0.0</param>
+        </state_interface>
       </joint>
-      <joint name="touch_z">
-        <command_interface name="effort"/>
-        <state_interface name="position"/>
-        <state_interface name="velocity"/>
+      <joint name="elbow">
+        <state_interface name="position">
+          <param name="initial_value">0.0</param>
+        </state_interface>
+        <state_interface name="velocity">
+          <param name="initial_value">0.0</param>
+        </state_interface>
       </joint>
+      <joint name="yaw">
+        <state_interface name="position">
+          <param name="initial_value">0.0</param>
+        </state_interface>
+        <state_interface name="velocity">
+          <param name="initial_value">0.0</param>
+        </state_interface>
+      </joint>
+      <joint name="pitch">
+        <state_interface name="position">
+          <param name="initial_value">0.0</param>
+        </state_interface>
+        <state_interface name="velocity">
+          <param name="initial_value">0.0</param>
+        </state_interface>
+      </joint>
+      <joint name="roll">
+        <state_interface name="position">
+          <param name="initial_value">0.0</param>
+        </state_interface>
+        <state_interface name="velocity">
+          <param name="initial_value">0.0</param>
+        </state_interface>
+      </joint>
+      <gpio name="force">
+        <command_interface name="force.x"/>
+        <command_interface name="force.y"/>
+        <command_interface name="force.z"/>
+        <state_interface name="force.x">
+          <param name="initial_value">0.0</param>
+        </state_interface>
+        <state_interface name="force.y">
+          <param name="initial_value">0.0</param>
+        </state_interface>
+        <state_interface name="force.z">
+          <param name="initial_value">0.0</param>
+        </state_interface>
+      </gpio>
+      <sensor name="tcp_pose">
+        <state_interface name="position.x">
+          <param name="initial_value">0.0</param>
+        </state_interface>
+        <state_interface name="position.y">
+          <param name="initial_value">0.0</param>
+        </state_interface>
+        <state_interface name="position.z">
+          <param name="initial_value">0.0</param>
+        </state_interface>
+        <state_interface name="orientation.x">
+          <param name="initial_value">0.0</param>
+        </state_interface>
+        <state_interface name="orientation.y">
+          <param name="initial_value">0.0</param>
+        </state_interface>
+        <state_interface name="orientation.z">
+          <param name="initial_value">0.0</param>
+        </state_interface>
+        <state_interface name="orientation.w">
+          <param name="initial_value">1.0</param>
+        </state_interface>
+        <param name="frame_id">touch_tcp</param>
+      </sensor>
     </ros2_control>
   </xacro:macro>

File: touch_description/urdf/touch.urdf.xacro (robot description, xacro)
@@ -4,34 +4,123 @@
   <xacro:arg name="device_name" default="Default Device"/>
   <xacro:include filename="$(find touch_description)/ros2_control/touch.ros2_control.xacro"/>
-  <link name="touch_base"/>
-  <link name="touch_x_link"/>
-  <link name="touch_y_link"/>
-  <link name="touch_z_link"/>
-  <link name="stylus_tip"/>
-  <joint name="touch_x" type="prismatic">
+  <material name="metal_seamed">
+    <color rgba="0.4627450980392157 0.4666666666666667 0.4509803921568628 1.0"/>
+  </material>
+  <material name="blue">
+    <color rgba="0.0 0.0 0.8 1.0"/>
+  </material>
+  <material name="white">
+    <color rgba="1.0 1.0 1.0 1.0"/>
+  </material>
+  <link name="touch_base">
+    <visual>
+      <origin xyz="0 -0.02 0"/>
+      <geometry>
+        <mesh filename="package://touch_description/meshes/base.stl"/>
+      </geometry>
+      <material name="metal_seamed"/>
+    </visual>
+  </link>
+  <link name="torso">
+    <visual>
+      <origin xyz="0 0 0.036" rpy="-1.5707 0 0"/>
+      <geometry>
+        <mesh filename="package://touch_description/meshes/torso.stl"/>
+      </geometry>
+      <material name="blue"/>
+    </visual>
+  </link>
+  <link name="upper_arm">
+    <visual>
+      <origin xyz="0.0075 0 0" rpy="0 0 0"/>
+      <geometry>
+        <mesh filename="package://touch_description/meshes/upper_arm.stl"/>
+      </geometry>
+      <material name="metal_seamed"/>
+    </visual>
+  </link>
+  <link name="lower_arm">
+    <visual>
+      <origin xyz="0 0 0" rpy="1.5707 0 0"/>
+      <geometry>
+        <mesh filename="package://touch_description/meshes/lower_arm.stl"/>
+      </geometry>
+      <material name="metal_seamed"/>
+    </visual>
+  </link>
+  <link name="wrist">
+    <visual>
+      <origin xyz="0 0 0" rpy="3.14159 0 0"/>
+      <geometry>
+        <mesh filename="package://touch_description/meshes/wrist.stl"/>
+      </geometry>
+      <material name="metal_seamed"/>
+    </visual>
+  </link>
+  <link name="tip">
+    <visual>
+      <origin xyz="0 0 0" rpy="-1.5707 0 0"/>
+      <geometry>
+        <mesh filename="package://touch_description/meshes/tip.stl"/>
+      </geometry>
+      <material name="metal_seamed"/>
+    </visual>
+  </link>
+  <link name="stylus">
+    <visual>
+      <origin xyz="0 -0.039 0" rpy="1.5707 1.5707 0"/>
+      <geometry>
+        <mesh filename="package://touch_description/meshes/stylus.stl"/>
+      </geometry>
+      <material name="blue"/>
+    </visual>
+  </link>
+  <link name="touch_tcp"/>
+  <joint name="waist" type="revolute">
     <parent link="touch_base"/>
-    <child link="touch_x_link"/>
-    <origin xyz="0 0 0" rpy="0 0 0"/>
+    <child link="torso"/>
+    <origin xyz="0 0 0.09" rpy="0 0 0"/>
+    <axis xyz="0 0 1"/>
+    <limit lower="-0.98" upper="0.98" velocity="100" effort="5"/>
+  </joint>
+  <joint name="shoulder" type="revolute">
+    <parent link="torso"/>
+    <child link="upper_arm"/>
+    <origin xyz="-0.0075 0 0.035" rpy="0 0 0"/>
     <axis xyz="1 0 0"/>
-    <limit effort="12.0" velocity="2.0" lower="-0.2" upper="0.2"/>
+    <limit lower="0" upper="1.75" velocity="100" effort="5"/>
   </joint>
-  <joint name="touch_y" type="prismatic">
-    <parent link="touch_x_link"/>
-    <child link="touch_y_link"/>
-    <origin xyz="0 0 0" rpy="0 0 0"/>
+  <joint name="elbow" type="revolute">
+    <parent link="upper_arm"/>
+    <child link="lower_arm"/>
+    <origin xyz="0.0075 0.134 0" rpy="-1.5 0 0"/>
+    <axis xyz="1 0 0"/>
+    <limit lower="-0.81" upper="1.25" velocity="100" effort="5"/>
+  </joint>
+  <joint name="yaw" type="revolute">
+    <parent link="lower_arm"/>
+    <child link="wrist"/>
+    <origin xyz="0 0.08 0" rpy="0 0 0"/>
     <axis xyz="0 1 0"/>
-    <limit effort="12.0" velocity="2.0" lower="-0.2" upper="0.2"/>
+    <limit lower="3.92" upper="8.83" velocity="100" effort="5"/>
   </joint>
-  <joint name="touch_z" type="prismatic">
-    <parent link="touch_y_link"/>
-    <child link="touch_z_link"/>
-    <origin xyz="0 0 0" rpy="0 0 0"/>
-    <axis xyz="0 0 1"/>
-    <limit effort="12.0" velocity="2.0" lower="-0.2" upper="0.2"/>
+  <joint name="pitch" type="revolute">
+    <parent link="wrist"/>
+    <child link="tip"/>
+    <origin xyz="0 0.0525 0" rpy="1.5707 0 0"/>
+    <axis xyz="1 0 0"/>
+    <limit lower="-0.5" upper="1.75" velocity="100" effort="5"/>
   </joint>
-  <joint name="stylus_tip_joint" type="fixed">
-    <parent link="touch_z_link"/>
-    <child link="stylus_tip"/>
-    <origin xyz="0 0 0" rpy="0 0 0"/>
+  <joint name="roll" type="revolute">
+    <parent link="tip"/>
+    <child link="stylus"/>
+    <origin xyz="0 -0.029 0" rpy="3.14159 3.14159 0"/>
+    <axis xyz="0 1 0"/>
+    <limit lower="-2.58" upper="2.58" velocity="100" effort="5"/>
+  </joint>
+  <joint name="tcp_joint" type="fixed">
+    <parent link="tip"/>
+    <child link="touch_tcp"/>
+    <origin xyz="0 0.031 0" rpy="0 0 0"/>
   </joint>
   <xacro:touch_ros2_control
